Commit message: quad final

File: body.urdf (robot description, URDF)
Before this commit: robot robot, 3 links, 2 joints
Links:
- added link BackFoot, mass 1; collision box size=0.2 0.2 1; visual box size=0.2 0.2 1
- added link FrontFoot, mass 1; collision box size=0.2 0.2 1; visual box size=0.2 0.2 1
- added link LeftFoot, mass 1; collision box size=0.2 0.2 1; visual box size=0.2 0.2 1
- added link LeftLeg, mass 1; collision box size=1 0.2 0.2; visual box size=1 0.2 0.2
- added link RightFoot, mass 1; collision box size=0.2 0.2 1; visual box size=0.2 0.2 1
- added link RightLeg, mass 1; collision box size=1 0.2 0.2; visual box size=1 0.2 0.2
- link BackLeg: geometry collision box size=0.2 1 0.2; visual box size=0.2 1 0.2
- link FrontLeg: geometry collision box size=0.2 1 0.2; visual box size=0.2 1 0.2
Joints:
- added joint BackKnee: type revolute, parent BackLeg, child BackFoot, origin xyz=0 -1 0 rpy=0 0 0, axis 1 1 0, limit lower=-3.14159 upper=3.14159 effort=0.0 velocity=0.0
- added joint FrontKnee: type revolute, parent FrontLeg, child FrontFoot, origin xyz=0 1 0 rpy=0 0 0, axis 1 1 0, limit lower=-3.14159 upper=3.14159 effort=0.0 velocity=0.0
- added joint LeftKnee: type revolute, parent LeftLeg, child LeftFoot, origin xyz=-1 0 0 rpy=0 0 0, axis 1 1 0, limit lower=-3.14159 upper=3.14159 effort=0.0 velocity=0.0
- added joint RightKnee: type revolute, parent RightLeg, child RightFoot, origin xyz=1 0 0 rpy=0 0 0, axis 1 1 0, limit lower=-3.14159 upper=3.14159 effort=0.0 velocity=0.0
- added joint Torso_LeftLeg: type revolute, parent Torso, child LeftLeg, origin xyz=-.5 0 1 rpy=0 0 0, axis 0 1 0, limit lower=-3.14159 upper=3.14159 effort=0.0 velocity=0.0
- added joint Torso_RightLeg: type revolute, parent Torso, child RightLeg, origin xyz=.5 0 1 rpy=0 0 0, axis 0 1 0, limit lower=-3.14159 upper=3.14159 effort=0.0 velocity=0.0
- joint Torso_BackLeg: axis 0 1 0 -> 1 0 0; origin xyz=.5 0 1 rpy=0 0 0 -> xyz=0 -.5 1 rpy=0 0 0
- joint Torso_FrontLeg: axis 0 1 0 -> 1 0 0; origin xyz=-.5 0 1 rpy=0 0 0 -> xyz=0 .5 1 rpy=0 0 0

Commit message: final

File: body.urdf (robot description, URDF)
Before this commit: robot robot, 9 links, 8 joints
Links:
- link BackFoot: geometry collision box size=0.2 0.2 1.8891930755260833; visual box size=0.2 0.2 1.8891930755260833
- link BackLeg: geometry collision box size=0.2 1.195695638480855 0.2; visual box size=0.2 1.195695638480855 0.2
- link FrontFoot: geometry collision box size=0.2 0.2 2.5792600906293144; visual box size=0.2 0.2 2.5792600906293144
- link FrontLeg: geometry collision box size=0.2 1.918659533324524 0.2; visual box size=0.2 1.918659533324524 0.2
- link LeftFoot: geometry collision box size=0.2 0.2 1.8555588600085762; visual box size=0.2 0.2 1.8555588600085762
- link LeftLeg: geometry collision box size=1.7009631131131626 0.2 0.2; visual box size=1.7009631131131626 0.2 0.2
- link RightFoot: geometry collision box size=0.2 0.2 0.6187519342517542; visual box size=0.2 0.2 0.6187519342517542
- link RightLeg: geometry collision box size=0.7099852270688949 0.2 0.2; visual box size=0.7099852270688949 0.2 0.2
Joints:
- joint BackKnee: origin xyz=0 -1 0 rpy=0 0 0 -> xyz=0 -1.195695638480855 0 rpy=0 0 0
- joint FrontKnee: origin xyz=0 1 0 rpy=0 0 0 -> xyz=0 1.918659533324524 0 rpy=0 0 0
- joint LeftKnee: origin xyz=-1 0 0 rpy=0 0 0 -> xyz=-1.7009631131131626 0 0 rpy=0 0 0
- joint RightKnee: origin xyz=1 0 0 rpy=0 0 0 -> xyz=0.7099852270688949 0 0 rpy=0 0 0
- joint Torso_BackLeg: origin xyz=0 -.5 1 rpy=0 0 0 -> xyz=0 -.5 5 rpy=0 0 0
- joint Torso_FrontLeg: origin xyz=0 .5 1 rpy=0 0 0 -> xyz=0 .5 5 rpy=0 0 0
- joint Torso_LeftLeg: origin xyz=-.5 0 1 rpy=0 0 0 -> xyz=-.5 0 5 rpy=0 0 0
- joint Torso_RightLeg: origin xyz=.5 0 1 rpy=0 0 0 -> xyz=.5 0 5 rpy=0 0 0
